File: Schema_circuit/Kicad/Projets/HM-Base/HM-Base.kicad_sch (KiCad schematic)
At the start: 25 parts, among them J1A1 Conn_01x02_Socket, J1B1 Conn_01x02_Pin, J2A1 Conn_01x02_Socket, J2B1 Conn_01x02_Pin, J3 Micro_SD_Card, J3A1 Conn_01x06_Socket, J4A1 Conn_01x06_Socket, J4B1 Conn_01x06_Pin, J5A1 Conn_01x08_Socket, J5B1 Conn_01x08_Pin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

Commit message: Rectification schema BASE
Parts:
- added D2: 1N4148, Diode_THT:D_DO-35_SOD27_P7.62mm_Horizontal, symbol Diode:1N4148
- J3: value Micro_SD_Card -> SD_Card
Connections:
- net at D1.1 (K), R3.2, U2.9 (EN): now also D2.1 (K); no longer R4.1, U3.J2-12 (IO14)
- net at R4.2: now also U3.J2-12 (IO14), D2.2 (A); no longer J3A1.5 (Pin_5)
- new net: J3A1.5 (Pin_5), R4.1
Other:
- note added: "Attention : retirer le strap sB2 sur le TPS63020 pour utiliser EN"
- company: (none) -> HumanLab
- title: (none) ->  INTERFACE ADAPTATIVE - Base
- moved on the sheet: D1, R4
Changed lines of the file:
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@@
 (kicad_sch (version 20230121) (generator eeschema)
   (paper "A4")
+  (title_block
+    (title " INTERFACE ADAPTATIVE - Base")
+    (date "2023-03-24")
+    (company "HumanLab")
+  )
   (junction (at 90.17 58.42) (diameter 0) (color 0 0 0 0)
   )
@@
   )
   (junction (at 111.76 97.79) (diameter 0) (color 0 0 0 0)
+  )
+  (junction (at 132.08 95.25) (diameter 0) (color 0 0 0 0)
   )
   (junction (at 86.36 83.82) (diameter 0) (color 0 0 0 0)
@@
     (stroke (width 0) (type default))
   )
-  (wire (pts (xy 111.76 97.79) (xy 124.46 97.79))
+  (wire (pts (xy 111.76 97.79) (xy 114.3 97.79))
     (stroke (width 0) (type default))
   )
@@
     (stroke (width 0) (type default))
   )
-  (wire (pts (xy 111.76 95.25) (xy 144.78 95.25))
-    (stroke (width 0) (type default))
-  )
-  (wire (pts (xy 111.76 138.43) (xy 111.76 107.95))
+  (wire (pts (xy 111.76 95.25) (xy 121.92 95.25))
+    (stroke (width 0) (type default))
+  )
+  (wire (pts (xy 111.76 107.95) (xy 111.76 138.43))
     (stroke (width 0) (type default))
   )
@@
   )
   (wire (pts (xy 142.24 67.31) (xy 144.78 67.31))
-    (stroke (width 0) (type default))
-  )
-  (wire (pts (xy 111.76 100.33) (xy 111.76 97.79))
     (stroke (width 0) (type default))
   )
@@
     (stroke (width 0) (type default))
   )
+  (wire (pts (xy 129.54 95.25) (xy 132.08 95.25))
+    (stroke (width 0) (type default))
+  )
   (wire (pts (xy 82.55 76.2) (xy 88.9 76.2))
     (stroke (width 0) (type default))
   )
+  (wire (pts (xy 123.19 107.95) (xy 132.08 107.95))
+    (stroke (width 0) (type default))
+  )
   (wire (pts (xy 116.84 132.08) (xy 116.84 138.43))
     (stroke (width 0) (type default))
@@
   )
   (wire (pts (xy 142.24 149.86) (xy 142.24 160.02))
+    (stroke (width 0) (type default))
+  )
+  (wire (pts (xy 115.57 107.95) (xy 111.76 107.95))
     (stroke (width 0) (type default))
   )
@@
     (stroke (width 0) (type default))
   )
+  (wire (pts (xy 132.08 95.25) (xy 144.78 95.25))
+    (stroke (width 0) (type default))
+  )
   (wire (pts (xy 228.6 60.96) (xy 234.95 60.96))
     (stroke (width 0) (type default))
@@
     (stroke (width 0) (type default))
   )
-  (wire (pts (xy 132.08 138.43) (xy 132.08 114.3))
-    (stroke (width 0) (type default))
-  )
   (wire (pts (xy 185.42 85.09) (xy 200.66 85.09))
     (stroke (width 0) (type default))
@@
     (stroke (width 0) (type default))
   )
+  (wire (pts (xy 132.08 107.95) (xy 132.08 95.25))
+    (stroke (width 0) (type default))
+  )
   (wire (pts (xy 205.74 72.39) (xy 205.74 90.17))
     (stroke (width 0) (type default))
@@
     (stroke (width 0) (type default))
   )
-  (wire (pts (xy 132.08 97.79) (xy 144.78 97.79))
+  (wire (pts (xy 121.92 97.79) (xy 144.78 97.79))
     (stroke (width 0) (type default))
   )
@@
   )
   (wire (pts (xy 224.79 73.66) (xy 224.79 67.31))
+    (stroke (width 0) (type default))
+  )
+  (wire (pts (xy 132.08 114.3) (xy 132.08 138.43))
     (stroke (width 0) (type default))
   )
@@
   (text "Extension" (at 134.62 181.61 0)
     (effects (font (size 1.27 1.27)) (justify left bottom))
+  )
+  (text "Attention : retirer le strap sB2 sur le TPS63020 pour utiliser EN"
+    (at 19.05 193.04 0)
+    (effects (font (size 1.27 1.27) (color 255 4 11 1)) (justify left bottom))
   )
   (text "Vers \nPlateau utilisateur" (at 107.95 151.13 0)
@@
         (path "/3e60e72a-84eb-422e-9134-19b80d5dd9d4"
           (reference "#PWR012") (unit 1)
+        )
+      )
+    )
+  )
+  (symbol (lib_id "Diode:1N4148") (at 125.73 95.25 0) (unit 1)
+    (in_bom yes) (on_board yes) (dnp no)
+    (property "Reference" "D2" (at 125.73 91.44 0)
+      (effects (font (size 1.27 1.27)))
+    )
+    (property "Value" "1N4148" (at 125.73 92.71 0)
+      (effects (font (size 1.27 1.27)))
+    )
+    (property "Footprint" "Diode_THT:D_DO-35_SOD27_P7.62mm_Horizontal" (at 125.73 95.25 0)
+      (effects (font (size 1.27 1.27)) hide)
+    )
+    (property "Datasheet" "https://assets.nexperia.com/documents/data-sheet/1N4148_1N4448.pdf" (at 125.73 95.25 0)
+      (effects (font (size 1.27 1.27)) hide)
+    )
+    (property "Sim.Device" "D" (at 125.73 95.25 0)
+      (effects (font (size 1.27 1.27)) hide)
+    )
+    (property "Sim.Pins" "1=K 2=A" (at 125.73 95.25 0)
+      (effects (font (size 1.27 1.27)) hide)
+    )
+    (pin "1")
+    (pin "2")
+    (instances
+      (project "HM-Base"
+        (path "/3e60e72a-84eb-422e-9134-19b80d5dd9d4"
+          (reference "D2") (unit 1)
         )
       )
@@
       (effects (font (size 1.27 1.27)))
     )
-    (property "Value" "Micro_SD_Card" (at 258.445 50.8 0)
+    (property "Value" "SD_Card" (at 258.445 50.8 0)
       (effects (font (size 1.27 1.27)))
     )
@@
     )
   )
-  (symbol (lib_id "Device:R") (at 111.76 104.14 0) (unit 1)
-    (in_bom yes) (on_board yes) (dnp no) (fields_autoplaced)
-    (property "Reference" "R4" (at 114.3 103.505 0)
-      (effects (font (size 1.27 1.27)) (justify left))
-    )
-    (property "Value" "330k" (at 114.3 106.045 0)
-      (effects (font (size 1.27 1.27)) (justify left))
-    )
-    (property "Footprint" "Resistor_THT:R_Axial_DIN0207_L6.3mm_D2.5mm_P10.16mm_Horizontal" (at 109.982 104.14 90)
-      (effects (font (size 1.27 1.27)) hide)
-    )
-    (property "Datasheet" "~" (at 111.76 104.14 0)
+  (symbol (lib_id "Device:R") (at 119.38 107.95 90) (unit 1)
+    (in_bom yes) (on_board yes) (dnp no)
+    (property "Reference" "R4" (at 119.38 104.14 90)
+      (effects (font (size 1.27 1.27)))
+    )
+    (property "Value" "330k" (at 119.38 105.41 90)
+      (effects (font (size 1.27 1.27)))
+    )
+    (property "Footprint" "Resistor_THT:R_Axial_DIN0207_L6.3mm_D2.5mm_P10.16mm_Horizontal" (at 119.38 109.728 90)
+      (effects (font (size 1.27 1.27)) hide)
+    )
+    (property "Datasheet" "~" (at 119.38 107.95 0)
       (effects (font (size 1.27 1.27)) hide)
     )
@@
     )
   )
-  (symbol (lib_id "Diode:1N4148") (at 128.27 97.79 0) (unit 1)
-    (in_bom yes) (on_board yes) (dnp no)
-    (property "Reference" "D1" (at 128.27 100.33 0)
-      (effects (font (size 1.27 1.27)))
-    )
-    (property "Value" "1N4148" (at 128.27 101.6 0)
-      (effects (font (size 1.27 1.27)))
-    )
-    (property "Footprint" "Diode_THT:D_DO-35_SOD27_P7.62mm_Horizontal" (at 128.27 97.79 0)
-      (effects (font (size 1.27 1.27)) hide)
-    )
-    (property "Datasheet" "https://assets.nexperia.com/documents/data-sheet/1N4148_1N4448.pdf" (at 128.27 97.79 0)
-      (effects (font (size 1.27 1.27)) hide)
-    )
-    (property "Sim.Device" "D" (at 128.27 97.79 0)
-      (effects (font (size 1.27 1.27)) hide)
-    )
-    (property "Sim.Pins" "1=K 2=A" (at 128.27 97.79 0)
-      (effects (font (size 1.27 1.27)) hide)
-    )
+  (symbol (lib_id "Diode:1N4148") (at 118.11 97.79 0) (unit 1)
+    (in_bom yes) (on_board yes) (dnp no)
+    (property "Reference" "D1" (at 118.11 100.33 0)
+      (effects (font (size 1.27 1.27)))
+    )
+    (property "Value" "1N4148" (at 118.11 101.6 0)
+      (effects (font (size 1.27 1.27)))
+    )
+    (property "Footprint" "Diode_THT:D_DO-35_SOD27_P7.62mm_Horizontal" (at 118.11 97.79 0)
+      (effects (font (size 1.27 1.27)) hide)
+    )
+    (property "Datasheet" "https://assets.nexperia.com/documents/data-sheet/1N4148_1N4448.pdf" (at 118.11 97.79 0)
+      (effects (font (size 1.27 1.27)) hide)
+    )
+    (property "Sim.Device" "D" (at 118.11 97.79 0)
+      (effects (font (size 1.27 1.27)) hide)
+    )
+    (property "Sim.Pins" "1=K 2=A" (at 118.11 97.79 0)
+      (effects (font (size 1.27 1.27)) hide)
+    )

Commit message: MaJ 29-04-23
Connections:
- net at U1.3 (Vout1), U2.1 (Vin1): now also J3A1.6 (Pin_6)
- net at R2.2, U1.4 (Bat+): now also J4A1.6 (Pin_6); no longer J4A1.5 (Pin_5)
- new net: J2A1.1 (Pin_1), J4A1.5 (Pin_5)
Other:
- moved on the sheet: BT1, J2A1, J2B1, J3A1, J4A1, J4B1, J7, R1, R2, R3, R4
